Commit message: fix(robot): stop derived assets from overwriting manifests or pinning dev paths
Three problems in the normalization path.

The manifest was written to a fixed normalization_manifest.json in the output
directory, so a second asset normalized into the same directory would silently
destroy the first one's provenance. It is now named after the artifact, the
returned dict reports where it went, and the gate proves two assets sharing a
directory keep both manifests.

The committed normalized Allegro URDF embedded 42 absolute paths from the machine
that produced it, which PLAN.md forbids and which makes the artifact unusable
anywhere else. URDF mesh references resolve relative to the model file, so the
package replacement is now relative to the output directory. Regenerated; MuJoCo
still loads it with nq=16. A gate check now scans every committed derived asset
for absolute paths.

sanitize_inertia_matrix only tested positive-definiteness and off-diagonal
dominance on the pass-through path. MuJoCo also rejects inertias that violate
A + B >= C, one of the errors this transform exists to repair, so the triangle
inequality is checked before passing a tensor through unchanged. No link in the
Allegro URDF hits the new branch -- the regenerated output is byte-identical
apart from the mesh paths.

Also corrected a comment claiming attributes were sorted; ElementTree keeps them
in document order, which is what makes the output reproducible.

Co-Authored-By: Claude Opus 5 <noreply@anthropic.com>

File: qdgrasp/assets/derived/allegro_hand_description_right_A.normalized.urdf (robot description, URDF)
Before this commit: robot allegro_hand_right, 22 links, 21 joints
Links:
- link link_0_0: geometry collision mesh filename=../../../.references/robot-assets/wonik-allegro-ros2/src/al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 scale=0.001 0.001 0.001; visual mesh filename=../../../.references/robot-assets/wonik-allegro-ros2/src/al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 scale=0.001 0.001 0.001
- link link_10_0: geometry collision mesh filename=../../../.references/robot-assets/wonik-allegro-ros2/src/al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 scale=0.001 0.001 0.001; visual mesh filename=../../../.references/robot-assets/wonik-allegro-ros2/src/al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 scale=0.001 0.001 0.001
- link link_11_0: geometry collision mesh filename=../../../.references/robot-assets/wonik-allegro-ros2/src/al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 scale=0.001 0.001 0.001; visual mesh filename=../../../.references/robot-assets/wonik-allegro-ros2/src/al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 scale=0.001 0.001 0.001
- link link_11_0_tip: geometry collision mesh filename=../../../.references/robot-assets/wonik-allegro-ros2/src/al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 scale=0.001 0.001 0.001; visual mesh filename=../../../.references/robot-assets/wonik-allegro-ros2/src/al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 scale=0.001 0.001 0.001
- link link_12_0: geometry collision mesh filename=../../../.references/robot-assets/wonik-allegro-ros2/src/al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 scale=0.001 0.001 0.001; visual mesh filename=../../../.references/robot-assets/wonik-allegro-ros2/src/al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 scale=0.001 0.001 0.001
- link link_13_0: geometry collision mesh filename=../../../.references/robot-assets/wonik-allegro-ros2/src/al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 scale=0.001 0.001 0.001; visual mesh filename=../../../.references/robot-assets/wonik-allegro-ros2/src/al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 scale=0.001 0.001 0.001
- link link_14_0: geometry collision mesh filename=../../../.references/robot-assets/wonik-allegro-ros2/src/al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 scale=0.001 0.001 0.001; visual mesh filename=../../../.references/robot-assets/wonik-allegro-ros2/src/al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 scale=0.001 0.001 0.001
- link link_15_0: geometry collision mesh filename=../../../.references/robot-assets/wonik-allegro-ros2/src/al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 scale=0.001 0.001 0.001; visual mesh filename=../../../.references/robot-assets/wonik-allegro-ros2/src/al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 scale=0.001 0.001 0.001
- link link_15_0_tip: geometry collision mesh filename=../../../.references/robot-assets/wonik-allegro-ros2/src/al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 scale=0.001 0.001 0.001; visual mesh filename=../../../.references/robot-assets/wonik-allegro-ros2/src/al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 scale=0.001 0.001 0.001
- link link_1_0: geometry collision mesh filename=../../../.references/robot-assets/wonik-allegro-ros2/src/al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 scale=0.001 0.001 0.001; visual mesh filename=../../../.references/robot-assets/wonik-allegro-ros2/src/al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 scale=0.001 0.001 0.001
- link link_2_0: geometry collision mesh filename=../../../.references/robot-assets/wonik-allegro-ros2/src/al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 scale=0.001 0.001 0.001; visual mesh filename=../../../.references/robot-assets/wonik-allegro-ros2/src/al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 scale=0.001 0.001 0.001
- link link_3_0: geometry collision mesh filename=../../../.references/robot-assets/wonik-allegro-ros2/src/al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 scale=0.001 0.001 0.001; visual mesh filename=../../../.references/robot-assets/wonik-allegro-ros2/src/al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 scale=0.001 0.001 0.001
- link link_3_0_tip: geometry collision mesh filename=../../../.references/robot-assets/wonik-allegro-ros2/src/al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 scale=0.001 0.001 0.001; visual mesh filename=../../../.references/robot-assets/wonik-allegro-ros2/src/al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 scale=0.001 0.001 0.001
- link link_4_0: geometry collision mesh filename=../../../.references/robot-assets/wonik-allegro-ros2/src/al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 scale=0.001 0.001 0.001; visual mesh filename=../../../.references/robot-assets/wonik-allegro-ros2/src/al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 scale=0.001 0.001 0.001
- link link_5_0: geometry collision mesh filename=../../../.references/robot-assets/wonik-allegro-ros2/src/al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 scale=0.001 0.001 0.001; visual mesh filename=../../../.references/robot-assets/wonik-allegro-ros2/src/al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 scale=0.001 0.001 0.001
- link link_6_0: geometry collision mesh filename=../../../.references/robot-assets/wonik-allegro-ros2/src/al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 scale=0.001 0.001 0.001; visual mesh filename=../../../.references/robot-assets/wonik-allegro-ros2/src/al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 scale=0.001 0.001 0.001
- link link_7_0: geometry collision mesh filename=../../../.references/robot-assets/wonik-allegro-ros2/src/al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 scale=0.001 0.001 0.001; visual mesh filename=../../../.references/robot-assets/wonik-allegro-ros2/src/al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 scale=0.001 0.001 0.001
- link link_7_0_tip: geometry collision mesh filename=../../../.references/robot-assets/wonik-allegro-ros2/src/al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 scale=0.001 0.001 0.001; visual mesh filename=../../../.references/robot-assets/wonik-allegro-ros2/src/al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 scale=0.001 0.001 0.001
- link link_8_0: geometry collision mesh filename=../../../.references/robot-assets/wonik-allegro-ros2/src/al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 scale=0.001 0.001 0.001; visual mesh filename=../../../.references/robot-assets/wonik-allegro-ros2/src/al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 scale=0.001 0.001 0.001
- link link_9_0: geometry collision mesh filename=../../../.references/robot-assets/wonik-allegro-ros2/src/al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 scale=0.001 0.001 0.001; visual mesh filename=../../../.references/robot-assets/wonik-allegro-ros2/src/al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 scale=0.001 0.001 0.001
- link palm_link: geometry collision mesh filename=../../../.references/robot-assets/wonik-allegro-ros2/src/al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 scale=0.001 0.001 0.001; visual mesh filename=../../../.references/robot-assets/wonik-allegro-ros2/src/al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 scale=0.001 0.001 0.001
